Commit message: Add gripper to simulation. (WIP)

File: ur_e_description/urdf/ur.gazebo.xacro (robot description, xacro)
@@ -23,4 +23,13 @@
       <selfCollide>true</selfCollide>
     </gazebo>
+    <gazebo reference="${prefix}gripper_link">
+      <selfCollide>true</selfCollide>
+    </gazebo>
+    <gazebo reference="${prefix}left_finger_link">
+      <selfCollide>true</selfCollide>
+    </gazebo>
+    <gazebo reference="${prefix}right_finger_link">
+      <selfCollide>true</selfCollide>
+    </gazebo>
   </xacro:macro>
 </robot>

File: ur_e_description/urdf/ur.transmission.xacro (robot description, xacro)
@@ -56,4 +56,24 @@
       </actuator>
     </transmission>
+    <transmission name="${prefix}left_finger_trans">
+      <type>transmission_interface/SimpleTransmission</type>
+      <joint name="${prefix}left_finger_joint">
+        <hardwareInterface>hardware_interface/PositionJointInterface</hardwareInterface>
+      </joint>
+      <actuator name="${prefix}left_finger_motor">
+        <hardwareInterface>hardware_interface/PositionJointInterface</hardwareInterface>
+        <mechanicalReduction>1</mechanicalReduction>
+      </actuator>
+    </transmission>
+    <transmission name="${prefix}right_finger_trans">
+      <type>transmission_interface/SimpleTransmission</type>
+      <joint name="${prefix}right_finger_joint">
+        <hardwareInterface>hardware_interface/PositionJointInterface</hardwareInterface>
+      </joint>
+      <actuator name="${prefix}right_finger_motor">
+        <hardwareInterface>hardware_interface/PositionJointInterface</hardwareInterface>
+        <mechanicalReduction>1</mechanicalReduction>
+      </actuator>
+    </transmission>
   </xacro:macro>
 </robot>

File: ur_e_description/urdf/ur10e.urdf.xacro (robot description, xacro)
@@ -321,4 +321,103 @@
       </collision>
     </link>
+    <link name="${prefix}gripper_link">
+        <visual>
+            <geometry>
+                <mesh filename="package://ur_e_description/meshes/ur10e/visual/weiss-mount.dae"/>
+            </geometry>
+            <origin xyz="-0.071 0 0" rpy="${pi/-2.0} 0 ${pi/-2.0}"/>
+        </visual>
+        <visual>
+            <geometry>
+                <mesh filename="package://ur_e_description/meshes/ur10e/visual/weiss-cg.dae"/>
+            </geometry>
+            <origin xyz="-0.07 0 0" rpy="${pi/-2.0} 0 ${pi/-2.0}"/>
+        </visual>
+        <collision>
+            <geometry>
+                <box size="0.071 0.105 0.06"/>
+            </geometry>
+            <origin rpy="0 0 0" xyz="${-0.071*0.5} 0 0"/>
+        </collision>
+        <inertial>
+            <origin xyz="0 0 0" rpy="0 0 0" />
+            <mass value="1.7" />
+            <inertia
+                ixx="1.0" ixy="0.0" ixz="0.0"
+                iyy="1.0" iyz="0.0"
+                izz="1.0" />
+        </inertial>
+      <dynamics damping="0.0" friction="0.0"/>
+    </link>
+    <joint name="${prefix}gripper_fixed_joint" type="fixed">
+        <origin xyz="0.071 0 0" rpy="0 0 0"/>
+        <parent link="${prefix}ee_link"/>
+        <child link="${prefix}gripper_link"/>
+    </joint>
+    <joint name="${prefix}left_finger_joint" type="prismatic">
+        <origin xyz="0 0.02 0" rpy="0 0 0"/>
+        <axis xyz="0 1 0"/>
+        <limit lower="0" upper="0.02" effort="100" velocity="0.05"/>
+        <parent link="${prefix}gripper_link"/>
+        <child link="${prefix}left_finger_link"/>
+    </joint>
+    <link name="${prefix}left_finger_link">
+        <visual>
+            <geometry>
+                <box size="0.095 0.02 0.02"/>
+            </geometry>
+            <material name="LightGrey">
+                <color rgba="0.7 0.7 0.7 1.0"/>
+            </material>
+            <origin xyz="${0.095*0.5} 0 0" rpy="0 0 0"/>
+        </visual>
+        <collision>
+            <geometry>
+                <box size="0.095 0.02 0.02"/>
+            </geometry>
+            <origin xyz="${0.095*0.5} 0 0" rpy="0 0 0"/>
+        </collision>
+        <inertial>
+            <origin xyz="0 0 0" rpy="0 0 0" />
+            <mass value="0.1" />
+            <inertia
+                ixx="1.0" ixy="0.0" ixz="0.0"
+                iyy="1.0" iyz="0.0"
+                izz="1.0" />
+        </inertial>
+    </link>
+    <link name="${prefix}right_finger_link">
+        <visual>
+            <geometry>
+                <box size="0.095 0.02 0.02"/>
+            </geometry>
+            <material name="LightGrey">
+                <color rgba="0.7 0.7 0.7 1.0"/>
+            </material>
+            <origin xyz="${0.095*0.5} 0 0" rpy="0 0 0"/>
+        </visual>
+        <collision>
+            <geometry>
+                <box size="0.095 0.02 0.02"/>
+            </geometry>
+            <origin xyz="${0.095*0.5} 0 0" rpy="0 0 0"/>
+        </collision>
+        <inertial>
+            <origin xyz="0 0 0" rpy="0 0 0" />
+            <mass value="0.1" />
+            <inertia
+                ixx="1.0" ixy="0.0" ixz="0.0"
+                iyy="1.0" iyz="0.0"
+                izz="1.0" />
+        </inertial>
+    </link>
+    <joint name="${prefix}right_finger_joint" type="prismatic">
+        <!-- <origin xyz="0 -0.0425 0" rpy="0 0 0"/> -->
+        <origin xyz="0 -0.02 0" rpy="0 0 0"/>
+        <axis xyz="0 -1 0"/>
+        <limit lower="0" upper="0.02" effort="100" velocity="0.05"/>
+        <parent link="${prefix}gripper_link"/>
+        <child link="${prefix}right_finger_link"/>
+    </joint>
     <xacro:ur_arm_transmission prefix="${prefix}" />
     <xacro:ur_arm_gazebo prefix="${prefix}" />
@@ -341,29 +440,4 @@
       <child link="${prefix}tool0"/>
     </joint>
-    <link name="${prefix}gripper_link">
-        <visual>
-            <geometry>
-                <mesh filename="package://ur_e_description/meshes/ur10e/visual/weiss-mount.dae"/>
-            </geometry>
-            <origin xyz="-0.071 0 0" rpy="${pi/-2.0} 0 ${pi/-2.0}"/>
-        </visual>
-        <visual>
-            <geometry>
-                <mesh filename="package://ur_e_description/meshes/ur10e/visual/weiss-cg.dae"/>
-            </geometry>
-            <origin xyz="-0.07 0 0" rpy="${pi/-2.0} 0 ${pi/-2.0}"/>
-        </visual>
-        <collision>
-            <geometry>
-                <box size="0.071 0.105 0.06"/>
-            </geometry>
-            <origin rpy="0 0 0" xyz="${0.071*0.5} 0 0"/>
-        </collision>
-    </link>
-    <joint name="${prefix}gripper_fixed_joint" type="fixed">
-        <origin xyz="0.071 0 0" rpy="0 0 0"/>
-        <parent link="${prefix}ee_link"/>
-        <child link="${prefix}gripper_link"/>
-    </joint>
   </xacro:macro>
 </robot>

Commit message: Add gripper driver (WIP). Add camera to gripper.

File: ur_e_description/urdf/ur.gazebo.xacro (robot description, xacro)
@@ -33,3 +33,41 @@
     </gazebo>
   </xacro:macro>
+  <xacro:macro name="sim_3dsensor" params="prefix">
+      <gazebo reference="${prefix}_rgb_frame">
+          <sensor type="depth" name="camera">
+              <always_on>true</always_on>
+              <update_rate>20.0</update_rate>
+              <camera>
+                  <horizontal_fov>${60.0*pi/180.0}</horizontal_fov>
+                  <image>
+                      <format>B8G8R8</format>
+                      <width>640</width>
+                      <height>480</height>
+                  </image>
+                  <clip>
+                      <near>0.10</near>
+                      <far>8.0</far>
+                  </clip>
+              </camera>
+              <plugin name="${prefix}_camera_controller" filename="libgazebo_ros_openni_kinect.so">
+                  <cameraName>${prefix}</cameraName>
+                  <alwaysOn>true</alwaysOn>
+                  <updateRate>10</updateRate>
+                  <imageTopicName>rgb/image_raw</imageTopicName>
+                  <depthImageTopicName>depth/image_raw</depthImageTopicName>
+                  <pointCloudTopicName>depth/points</pointCloudTopicName>
+                  <cameraInfoTopicName>rgb/camera_info</cameraInfoTopicName>
+                  <depthImageCameraInfoTopicName>depth/camera_info</depthImageCameraInfoTopicName>
+                  <frameName>${prefix}_depth_optical_frame</frameName>
+                  <baseline>0.1</baseline>
+                  <distortion_k1>0.0</distortion_k1>
+                  <distortion_k2>0.0</distortion_k2>
+                  <distortion_k3>0.0</distortion_k3>
+                  <distortion_t1>0.0</distortion_t1>
+                  <distortion_t2>0.0</distortion_t2>
+                  <pointCloudCutoff>0.4</pointCloudCutoff>
+              </plugin>
+          </sensor>
+      </gazebo>
+  </xacro:macro>
 </robot>

File: ur_e_description/urdf/ur10e.urdf.xacro (robot description, xacro)
@@ -358,5 +358,5 @@
         <origin xyz="0 0.02 0" rpy="0 0 0"/>
         <axis xyz="0 1 0"/>
-        <limit lower="0" upper="0.02" effort="100" velocity="0.05"/>
+        <limit lower="0" upper="0.03078" effort="100" velocity="0.05"/>
         <parent link="${prefix}gripper_link"/>
         <child link="${prefix}left_finger_link"/>
@@ -416,5 +416,5 @@
         <origin xyz="0 -0.02 0" rpy="0 0 0"/>
         <axis xyz="0 -1 0"/>
-        <limit lower="0" upper="0.02" effort="100" velocity="0.05"/>
+        <limit lower="0" upper="0.03078" effort="100" velocity="0.05"/>
         <parent link="${prefix}gripper_link"/>
         <child link="${prefix}right_finger_link"/>

File: ur_e_description/urdf/ur10e_joint_limited_robot.urdf.xacro (robot description, xacro)
@@ -15,4 +15,10 @@
 		 wrist_3_lower_limit="${-pi}" wrist_3_upper_limit="${pi}"
 />
+  <!-- sensor -->
+  <xacro:include filename="$(find ur_e_description)/urdf/astra.urdf.xacro" />
+  <xacro:sensor_astra parent="ee_link" prefix="camera">
+      <origin xyz="0.041311319304504816 -0.06402544453787727 0.044527571211305426"
+              rpy="3.13766148064 -0.00787797070144 0.000110993634886"/>
+  </xacro:sensor_astra>
   <link name="world" />
   <joint name="world_joint" type="fixed">

File: ur_e_description/urdf/ur10e_robot.urdf.xacro (robot description, xacro)
@@ -8,4 +8,9 @@
   <!-- arm -->
   <xacro:ur10e_robot prefix="" joint_limited="false"/>
+  <!-- sensor -->
+  <xacro:include filename="$(find ur_e_description)/urdf/astra.urdf.xacro" />
+  <xacro:sensor_astra parent="ee_link" prefix="camera">
+      <origin xyz="0.041311319304504816 -0.06402544453787727 0.044527571211305426" rpy="3.13766148064 -0.00787797070144 0.000110993634886"/>
+  </xacro:sensor_astra>
   <link name="world" />
   <joint name="world_joint" type="fixed">
